Commit message: Modifications for robot_walker and gazebo

File: urdf/one_legged_robot_walker.urdf (robot description, URDF)
Before this commit: robot one_legged_robot_walker, 7 links, 6 joints
Links:
- removed link map
Joints:
- removed joint body

File: urdf/robot_walker.urdf (robot description, URDF)
Before this commit: robot robot_walker, 7 links, 6 joints
Links:
- removed link map
- added link carpal_left_Tertiary; visual cylinder length=0.25 radius=0.065
- added link carpal_left_secondary; visual cylinder length=0.25 radius=0.065
- added link carpal_right_Tertiary; visual cylinder length=0.25 radius=0.065
- added link carpal_right_primary; visual cylinder length=0.25 radius=0.065
- added link carpal_right_secondary; visual cylinder length=0.25 radius=0.065
- added link foot_left_Tertiary; visual box size=0.2 0.2 0.05
- added link foot_left_secondary; visual box size=0.2 0.2 0.05
- added link foot_right_Tertiary; visual box size=0.2 0.2 0.05
- added link foot_right_primary; visual box size=0.2 0.2 0.05
- added link foot_right_secondary; visual box size=0.2 0.2 0.05
- added link humerus_left_Tertiary; visual cylinder length=0.85 radius=0.065
- added link humerus_left_secondary; visual cylinder length=0.85 radius=0.065
- added link humerus_right_Tertiary; visual cylinder length=0.85 radius=0.065
- added link humerus_right_primary; visual cylinder length=0.85 radius=0.065
- added link humerus_right_secondary; visual cylinder length=0.85 radius=0.065
- added link pectoral_left_Tertiary; visual box size=0.2 0.1 0.25
- added link pectoral_left_secondary; visual box size=0.2 0.1 0.25
- added link pectoral_right_Tertiary; visual box size=0.2 0.1 0.25
- added link pectoral_right_primary; visual box size=0.2 0.1 0.25
- added link pectoral_right_secondary; visual box size=0.2 0.1 0.25
- added link radius_left_Tertiary; visual cylinder length=0.45 radius=0.065
- added link radius_left_secondary; visual cylinder length=0.45 radius=0.065
- added link radius_right_Tertiary; visual cylinder length=0.45 radius=0.065
- added link radius_right_primary; visual cylinder length=0.45 radius=0.065
- added link radius_right_secondary; visual cylinder length=0.45 radius=0.065
Joints:
- removed joint body
- added joint pl_carpal_Tertiary: type revolute, parent radius_left_Tertiary, child carpal_left_Tertiary, origin xyz=0 0 -0.325, axis 0 1 0, limit lower=-1 upper=0 effort=1000.0 velocity=0.5
- added joint pl_carpal_right: type revolute, parent radius_right_primary, child carpal_right_primary, origin xyz=0 0 -0.325, axis 0 1 0, limit lower=-1 upper=0 effort=1000.0 velocity=0.5
- added joint pl_carpal_right_Tertiary: type revolute, parent radius_right_Tertiary, child carpal_right_Tertiary, origin xyz=0 0 -0.325, axis 0 1 0, limit lower=-1 upper=0 effort=1000.0 velocity=0.5
- added joint pl_carpal_right_secondary: type revolute, parent radius_right_secondary, child carpal_right_secondary, origin xyz=0 0 -0.325, axis 0 1 0, limit lower=-1 upper=0 effort=1000.0 velocity=0.5
- added joint pl_carpal_secondary: type revolute, parent radius_left_secondary, child carpal_left_secondary, origin xyz=0 0 -0.325, axis 0 1 0, limit lower=-1 upper=0 effort=1000.0 velocity=0.5
- added joint pl_foot_Tertiary: type revolute, parent carpal_left_Tertiary, child foot_left_Tertiary, origin xyz=0 0 -0.2, axis 0 1 0, limit lower=-1 upper=0 effort=1000.0 velocity=0.5
- added joint pl_foot_right: type revolute, parent carpal_right_primary, child foot_right_primary, origin xyz=0 0 -0.2, axis 0 1 0, limit lower=-1 upper=0 effort=1000.0 velocity=0.5
- added joint pl_foot_right_Tertiary: type revolute, parent carpal_right_Tertiary, child foot_right_Tertiary, origin xyz=0 0 -0.2, axis 0 1 0, limit lower=-1 upper=0 effort=1000.0 velocity=0.5
- added joint pl_foot_right_secondary: type revolute, parent carpal_right_secondary, child foot_right_secondary, origin xyz=0 0 -0.2, axis 0 1 0, limit lower=-1 upper=0 effort=1000.0 velocity=0.5
- added joint pl_foot_secondary: type revolute, parent carpal_left_secondary, child foot_left_secondary, origin xyz=0 0 -0.2, axis 0 1 0, limit lower=-1 upper=0 effort=1000.0 velocity=0.5
- added joint pl_humerus_Tertiary: type revolute, parent pectoral_left_Tertiary, child humerus_left_Tertiary, origin xyz=0 0.05 0, axis 0 1 0, limit lower=-1 upper=1 effort=1000.0 velocity=0.5
- added joint pl_humerus_right: type revolute, parent pectoral_right_primary, child humerus_right_primary, origin xyz=0 -0.05 0, axis 0 1 0, limit lower=-1 upper=1 effort=1000.0 velocity=0.5
- added joint pl_humerus_right_Tertiary: type revolute, parent pectoral_right_Tertiary, child humerus_right_Tertiary, origin xyz=0 -0.05 0, axis 0 1 0, limit lower=-1 upper=1 effort=1000.0 velocity=0.5
- added joint pl_humerus_right_secondary: type revolute, parent pectoral_right_secondary, child humerus_right_secondary, origin xyz=0 -0.05 0, axis 0 1 0, limit lower=-1 upper=1 effort=1000.0 velocity=0.5
- added joint pl_humerus_secondary: type revolute, parent pectoral_left_secondary, child humerus_left_secondary, origin xyz=0 0.05 0, axis 0 1 0, limit lower=-1 upper=1 effort=1000.0 velocity=0.5
- added joint pl_pectoral_Tertiary: type revolute, parent base_link, child pectoral_left_Tertiary, origin xyz=-0.8 0.5 0, axis 1 0 0, limit lower=0 upper=1 effort=1000.0 velocity=0.5
- added joint pl_pectoral_right: type revolute, parent base_link, child pectoral_right_primary, origin xyz=0.8 -0.5 0, axis 1 0 0, limit lower=-1 upper=0 effort=1000.0 velocity=0.5
- added joint pl_pectoral_right_Tertiary: type revolute, parent base_link, child pectoral_right_Tertiary, origin xyz=-0.8 -0.5 0, axis 1 0 0, limit lower=-1 upper=0 effort=1000.0 velocity=0.5
- added joint pl_pectoral_right_secondary: type revolute, parent base_link, child pectoral_right_secondary, origin xyz=0.15 -0.5 0, axis 1 0 0, limit lower=-1 upper=0 effort=1000.0 velocity=0.5
- added joint pl_pectoral_secondary: type revolute, parent base_link, child pectoral_left_secondary, origin xyz=0.15 0.5 0, axis 1 0 0, limit lower=0 upper=1 effort=1000.0 velocity=0.5
- added joint pl_radius_Tertiary: type revolute, parent humerus_left_Tertiary, child radius_left_Tertiary, origin xyz=0 0 -0.875, axis 0 1 0, limit lower=-1 upper=0 effort=1000.0 velocity=0.5
- added joint pl_radius_right: type revolute, parent humerus_right_primary, child radius_right_primary, origin xyz=0 0 -0.875, axis 0 1 0, limit lower=-1 upper=0 effort=1000.0 velocity=0.5
- added joint pl_radius_right_Tertiary: type revolute, parent humerus_right_Tertiary, child radius_right_Tertiary, origin xyz=0 0 -0.875, axis 0 1 0, limit lower=-1 upper=0 effort=1000.0 velocity=0.5
- added joint pl_radius_right_secondary: type revolute, parent humerus_right_secondary, child radius_right_secondary, origin xyz=0 0 -0.875, axis 0 1 0, limit lower=-1 upper=0 effort=1000.0 velocity=0.5
- added joint pl_radius_secondary: type revolute, parent humerus_left_secondary, child radius_left_secondary, origin xyz=0 0 -0.875, axis 0 1 0, limit lower=-1 upper=0 effort=1000.0 velocity=0.5
